Commit message: .

File: Robotics/URDF_Learning/3link.urdf (robot description, URDF)
Before this commit: robot pi_robot, 7 links, 6 joints
Links:
- link arm_1: geometry collision box size=.05 .3 .05; visual box size=.05 .3 .05
- link arm_2: geometry collision box size=.05 .3 .05; visual box size=.05 .3 .05
- link arm_3: geometry collision box size=.05 .3 .05; visual box size=.05 .3 .05
- link base: geometry collision cylinder length=.1 radius=0.1; visual cylinder length=.1 radius=0.1
- link base_cylinder: geometry collision cylinder length=.1 radius=0.05; visual cylinder length=.1 radius=0.05
- link second_cylinder: geometry collision cylinder length=.1 radius=0.05; visual cylinder length=.1 radius=0.05
- link third_cylinder: geometry collision cylinder length=.1 radius=0.05; visual cylinder length=.1 radius=0.05
Joints:
- joint base_joint: limit (none) -> lower=-1.57 upper=1.57 effort=10 velocity=3
- joint joint_arm1_c2: limit (none) -> lower=-1.57 upper=1.57 effort=10 velocity=3
- joint joint_arm2_c3: limit (none) -> lower=-1.57 upper=1.57 effort=10 velocity=3
- joint joint_c1_arm1: limit (none) -> lower=-1.57 upper=1.57 effort=10 velocity=3
- joint joint_c2_arm2: limit (none) -> lower=-1.57 upper=1.57 effort=10 velocity=3
- joint joint_c3_arm3: limit (none) -> lower=-1.57 upper=1.57 effort=10 velocity=3
