Commit message: .

File: Robotics/Pybullet_Workspace/Fig2_21_Parallelogram_arm.urdf (robot description, URDF)
Before this commit: robot parralelogram_arm, 10 links, 9 joints
Joints:
- joint joint_c1_arm1_prime: origin xyz=0.15 0 -> xyz=0.15 0 0

Commit message: .

File: Robotics/Pybullet_Workspace/Fig2_21_Parallelogram_arm.urdf (robot description, URDF)
Before this commit: robot parralelogram_arm, 10 links, 9 joints
Links:
- added link arm_4; collision box size=.05 .3 .05; visual box size=.05 .3 .05
- added link forth_cylinder_prime; collision cylinder length=.1 radius=0.05; visual cylinder length=.1 radius=0.04
Joints:
- removed joint joint_c1_arm1_prime
- added joint joint_arm_prime_c4_prime: type revolute, parent arm_1_prime, child forth_cylinder_prime, origin xyz=.15 0 0 rpy=0 0 0, axis 0 0 1, limit lower=-1.57 upper=1.57 effort=10 velocity=3
- added joint joint_c1_prime_arm1_prime: type fixed, parent first_cylinder_prime, child arm_1_prime, origin xyz=0.15 0 0, limit lower=-1.57 upper=1.57 effort=10 velocity=3
- added joint joint_c4_arm4: type fixed, parent forth_cylinder, child arm_4, origin xyz=0 .15 0
- joint joint_arm1_c2: limit lower=-1.57 upper=1.57 effort=10 velocity=3 -> lower=0 upper=1.57 effort=10 velocity=3; origin xyz=0 .15 0 -> xyz=0 .15 0 rpy=0 0 -1.57
- joint joint_arm2_c3: limit lower=-1.57 upper=1.57 effort=10 velocity=3 -> lower=0 upper=1.57 effort=10 velocity=3; origin xyz=0 .15 0 -> xyz=0 .15 0 rpy=0 0 -1.57
- joint joint_arm3_c4: origin xyz=0 .15 0 -> xyz=0 .15 0 rpy=0 0 0
- joint joint_c2_arm2: limit lower=-1.57 upper=1.57 effort=10 velocity=3 -> (none)
- joint joint_c3_arm3: limit lower=-1.57 upper=1.57 effort=10 velocity=3 -> (none)

Commit message: .

File: Robotics/Pybullet_Workspace/Fig2_21_Parallelogram_arm.urdf (robot description, URDF)
Before this commit: robot parralelogram_arm, 12 links, 11 joints
Joints:
- joint joint_arm3_c4: limit lower=-1.57 upper=1.57 effort=10 velocity=3 -> (none); type revolute -> fixed
- joint joint_arm_prime_c4_prime: limit lower=-1.57 upper=1.57 effort=10 velocity=3 -> (none); type revolute -> fixed
